File: _Electrical/BLE_REMOTE/BLEC_power.kicad_sch (KiCad schematic)
At the start: 19 parts, among them J6 LED, U2 BQ24232RGTR, U3 MIC5528-3.3YMX-TR

Commit message: JLCPCB parts selected
Parts:
- D1, D2: JLCPCB Part# (none) -> C2286; LCSC Part # (none) -> C2286; Part LS L29K-G1J2-1-Z -> KT-0603R
Changed lines of the file:
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@@
+      (effects (font (size 1.27 1.27)) hide)
+    )
+    (property "JLCPCB Part#" "" (at 64.77 114.3 0)
+      (effects (font (size 1.27 1.27)) hide)
+    )
+    (property "LCSC Part #" "" (at 64.77 114.3 0)
       (effects (font (size 1.27 1.27)) hide)
     )
@@
     )
     (property "Part" "RC0402JR-070RL" (at 59.69 109.22 0)
+      (effects (font (size 1.27 1.27)) hide)
+    )
+    (property "JLCPCB Part#" "" (at 59.69 109.22 0)
+      (effects (font (size 1.27 1.27)) hide)
+    )
+    (property "LCSC Part #" "" (at 59.69 109.22 0)
       (effects (font (size 1.27 1.27)) hide)
     )
@@
       (effects (font (size 1.27 1.27)) hide)
     )
+    (property "JLCPCB Part#" "" (at 143.51 66.04 0)
+      (effects (font (size 1.27 1.27)) hide)
+    )
+    (property "LCSC Part #" "" (at 143.51 66.04 0)
+      (effects (font (size 1.27 1.27)) hide)
+    )
     (pin "1")
     (pin "2")
@@
       (effects (font (size 1.27 1.27)) hide)
     )
+    (property "JLCPCB Part#" "" (at 45.72 68.58 0)
+      (effects (font (size 1.27 1.27)) hide)
+    )
+    (property "LCSC Part #" "" (at 45.72 68.58 0)
+      (effects (font (size 1.27 1.27)) hide)
+    )
     (pin "1")
     (pin "2")
@@
       (effects (font (size 1.27 1.27)) hide)
     )
+    (property "JLCPCB Part#" "" (at 54.61 104.14 0)
+      (effects (font (size 1.27 1.27)) hide)
+    )
+    (property "LCSC Part #" "" (at 54.61 104.14 0)
+      (effects (font (size 1.27 1.27)) hide)
+    )
     (pin "1")
     (pin "2")
@@
     )
     (property "Part" "ERJ-2RKF2001X" (at 134.62 69.85 0)
+      (effects (font (size 1.27 1.27)) hide)
+    )
+    (property "JLCPCB Part#" "" (at 134.62 69.85 0)
+      (effects (font (size 1.27 1.27)) hide)
+    )
+    (property "LCSC Part #" "" (at 134.62 69.85 0)
       (effects (font (size 1.27 1.27)) hide)
     )
@@
     )
     (property "Part" "MIC5528-3.3YMX-TR" (at 222.25 67.31 0)
+      (effects (font (size 1.27 1.27)) hide)
+    )
+    (property "JLCPCB Part#" "" (at 222.25 64.77 0)
+      (effects (font (size 1.27 1.27)) hide)
+    )
+    (property "LCSC Part #" "" (at 222.25 64.77 0)
       (effects (font (size 1.27 1.27)) hide)
     )
@@
       (effects (font (size 1.27 1.27)) hide)
     )
+    (property "JLCPCB Part#" "" (at 176.53 67.31 0)
+      (effects (font (size 1.27 1.27)) hide)
+    )
+    (property "LCSC Part #" "" (at 176.53 67.31 0)
+      (effects (font (size 1.27 1.27)) hide)
+    )
     (pin "1")
     (pin "2")
@@
       (effects (font (size 1.27 1.27)) hide)
     )
-    (property "Part" "LS L29K-G1J2-1-Z" (at 134.62 76.2 0)
+    (property "Part" "KT-0603R" (at 134.62 76.2 0)
+      (effects (font (size 1.27 1.27)) hide)
+    )
+    (property "JLCPCB Part#" "C2286" (at 134.62 76.2 0)
+      (effects (font (size 1.27 1.27)) hide)
+    )
+    (property "LCSC Part #" "C2286" (at 134.62 76.2 0)
       (effects (font (size 1.27 1.27)) hide)
     )
@@
     )
     (property "Part" "RC0402JR-0710KL" (at 135.89 100.33 0)
+      (effects (font (size 1.27 1.27)) hide)
+    )
+    (property "JLCPCB Part#" "" (at 135.89 100.33 0)
+      (effects (font (size 1.27 1.27)) hide)
+    )
+    (property "LCSC Part #" "" (at 135.89 100.33 0)
       (effects (font (size 1.27 1.27)) hide)
     )
@@
       (effects (font (size 1.27 1.27)) hide)
     )
+    (property "JLCPCB Part#" "" (at 102.87 163.83 0)
+      (effects (font (size 1.27 1.27)) hide)
+    )
+    (property "LCSC Part #" "" (at 102.87 163.83 0)
+      (effects (font (size 1.27 1.27)) hide)
+    )
     (pin "1")
     (pin "2")
@@
       (effects (font (size 1.27 1.27)) hide)
     )
+    (property "JLCPCB Part#" "" (at 45.72 91.44 0)
+      (effects (font (size 1.27 1.27)) hide)
+    )
+    (property "LCSC Part #" "" (at 45.72 91.44 0)
+      (effects (font (size 1.27 1.27)) hide)
+    )
     (pin "1")
     (pin "2")
@@
     )
     (property "Part" "RC0402FR-072K94L" (at 41.91 86.36 0)
+      (effects (font (size 1.27 1.27)) hide)
+    )
+    (property "JLCPCB Part#" "" (at 41.91 86.36 0)
+      (effects (font (size 1.27 1.27)) hide)
+    )
+    (property "LCSC Part #" "" (at 41.91 86.36 0)
       (effects (font (size 1.27 1.27)) hide)
     )
@@
       (effects (font (size 1.27 1.27)) hide)
     )
+    (property "JLCPCB Part#" "" (at 123.19 69.85 0)
+      (effects (font (size 1.27 1.27)) hide)
+    )
+    (property "LCSC Part #" "" (at 123.19 69.85 0)
+      (effects (font (size 1.27 1.27)) hide)
+    )
     (pin "1")
     (pin "2")
@@
     )
     (property "Part" "BQ24232RGTR" (at 95.25 92.71 0)
+      (effects (font (size 1.27 1.27)) hide)
+    )
+    (property "JLCPCB Part#" "" (at 95.25 92.71 0)
+      (effects (font (size 1.27 1.27)) hide)
+    )
+    (property "LCSC Part #" "" (at 95.25 92.71 0)
       (effects (font (size 1.27 1.27)) hide)
     )
@@
       (effects (font (size 1.27 1.27)) hide)
     )
-    (property "Part" "LS L29K-G1J2-1-Z" (at 123.19 76.2 0)
+    (property "Part" "KT-0603R" (at 123.19 76.2 0)
+      (effects (font (size 1.27 1.27)) hide)
+    )
+    (property "JLCPCB Part#" "C2286" (at 123.19 76.2 0)
+      (effects (font (size 1.27 1.27)) hide)
+    )
+    (property "LCSC Part #" "C2286" (at 123.19 76.2 0)
       (effects (font (size 1.27 1.27)) hide)
     )
@@
       (effects (font (size 1.27 1.27)) hide)
     )
+    (property "JLCPCB Part#" "" (at 226.06 67.31 0)
+      (effects (font (size 1.27 1.27)) hide)
+    )
+    (property "LCSC Part #" "" (at 226.06 67.31 0)
+      (effects (font (size 1.27 1.27)) hide)
+    )
     (pin "1")
     (pin "2")
@@
       (effects (font (size 1.27 1.27)) hide)
     )
+    (property "JLCPCB Part#" "" (at 49.53 99.06 0)
+      (effects (font (size 1.27 1.27)) hide)
+    )
+    (property "LCSC Part #" "" (at 49.53 99.06 0)
+      (effects (font (size 1.27 1.27)) hide)
+    )
     (pin "1")
     (pin "2")
@@
       (effects (font (size 1.27 1.27)) hide)
     )
+    (property "JLCPCB Part#" "" (at 59.69 76.2 0)
+      (effects (font (size 1.27 1.27)) hide)
+    )
+    (property "LCSC Part #" "" (at 59.69 76.2 0)
+      (effects (font (size 1.27 1.27)) hide)
+    )

Commit message: Adjusted components and changed buttons
Parts:
- renumbered C11 to C15, C12 to C16, C13 to C17, C14 to C18, J6 to J3
Changed lines of the file:
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@@
   (symbol (lib_id "power:+5V") (at 45.72 64.77 0) (unit 1)
     (in_bom yes) (on_board yes) (dnp no) (fields_autoplaced)
-    (property "Reference" "#PWR013" (at 45.72 68.58 0)
+    (property "Reference" "#PWR014" (at 45.72 68.58 0)
       (effects (font (size 1.27 1.27)) hide)
     )
@@
       (project "BLE_REMOTE"
         (path "/3c7105d6-b2e1-4841-966d-0562ae88783f/df7514b4-387c-47b1-a1bd-e93660408c5b"
-          (reference "#PWR013") (unit 1)
+          (reference "#PWR014") (unit 1)
         )
       )
@@
   (symbol (lib_id "power:+5V") (at 97.79 161.29 0) (unit 1)
     (in_bom yes) (on_board yes) (dnp no) (fields_autoplaced)
-    (property "Reference" "#PWR039" (at 97.79 165.1 0)
+    (property "Reference" "#PWR017" (at 97.79 165.1 0)
       (effects (font (size 1.27 1.27)) hide)
     )
@@
       (project "BLE_REMOTE"
         (path "/3c7105d6-b2e1-4841-966d-0562ae88783f/df7514b4-387c-47b1-a1bd-e93660408c5b"
-          (reference "#PWR039") (unit 1)
+          (reference "#PWR017") (unit 1)
         )
       )
@@
   (symbol (lib_id "power:GND") (at 226.06 76.2 0) (unit 1)
     (in_bom yes) (on_board yes) (dnp no)
-    (property "Reference" "#PWR021" (at 226.06 82.55 0)
+    (property "Reference" "#PWR022" (at 226.06 82.55 0)
       (effects (font (size 1.27 1.27)) hide)
     )
@@
       (project "BLE_REMOTE"
         (path "/3c7105d6-b2e1-4841-966d-0562ae88783f/df7514b4-387c-47b1-a1bd-e93660408c5b"
-          (reference "#PWR021") (unit 1)
+          (reference "#PWR022") (unit 1)
         )
       )
@@
   (symbol (lib_id "Device:C") (at 143.51 66.04 0) (unit 1)
     (in_bom yes) (on_board yes) (dnp no) (fields_autoplaced)
-    (property "Reference" "C12" (at 147.32 64.77 0)
+    (property "Reference" "C16" (at 147.32 64.77 0)
       (effects (font (size 1.27 1.27)) (justify left))
     )
@@
       (project "BLE_REMOTE"
         (path "/3c7105d6-b2e1-4841-966d-0562ae88783f/df7514b4-387c-47b1-a1bd-e93660408c5b"
-          (reference "C12") (unit 1)
+          (reference "C16") (unit 1)
         )
       )
@@
   (symbol (lib_id "power:VDD") (at 226.06 62.23 0) (unit 1)
     (in_bom yes) (on_board yes) (dnp no) (fields_autoplaced)
-    (property "Reference" "#PWR020" (at 226.06 66.04 0)
+    (property "Reference" "#PWR021" (at 226.06 66.04 0)
       (effects (font (size 1.27 1.27)) hide)
     )
@@
       (project "BLE_REMOTE"
         (path "/3c7105d6-b2e1-4841-966d-0562ae88783f/df7514b4-387c-47b1-a1bd-e93660408c5b"
+          (reference "#PWR021") (unit 1)
+        )
+      )
+    )
+  )
+  (symbol (lib_id "power:GND") (at 125.73 113.03 0) (unit 1)
+    (in_bom yes) (on_board yes) (dnp no) (fields_autoplaced)
+    (property "Reference" "#PWR020" (at 125.73 119.38 0)
+      (effects (font (size 1.27 1.27)) hide)
+    )
+    (property "Value" "GND" (at 125.73 118.11 0)
+      (effects (font (size 1.27 1.27)))
+    )
+    (property "Footprint" "" (at 125.73 113.03 0)
+      (effects (font (size 1.27 1.27)) hide)
+    )
+    (property "Datasheet" "" (at 125.73 113.03 0)
+      (effects (font (size 1.27 1.27)) hide)
+    )
+    (pin "1")
+    (instances
+      (project "BLE_REMOTE"
+        (path "/3c7105d6-b2e1-4841-966d-0562ae88783f/df7514b4-387c-47b1-a1bd-e93660408c5b"
           (reference "#PWR020") (unit 1)
         )
@@
     )
   )
-  (symbol (lib_id "power:GND") (at 125.73 113.03 0) (unit 1)
-    (in_bom yes) (on_board yes) (dnp no) (fields_autoplaced)
-    (property "Reference" "#PWR019" (at 125.73 119.38 0)
-      (effects (font (size 1.27 1.27)) hide)
-    )
-    (property "Value" "GND" (at 125.73 118.11 0)
-      (effects (font (size 1.27 1.27)))
-    )
-    (property "Footprint" "" (at 125.73 113.03 0)
-      (effects (font (size 1.27 1.27)) hide)
-    )
-    (property "Datasheet" "" (at 125.73 113.03 0)
-      (effects (font (size 1.27 1.27)) hide)
-    )
-    (pin "1")
-    (instances
-      (project "BLE_REMOTE"
-        (path "/3c7105d6-b2e1-4841-966d-0562ae88783f/df7514b4-387c-47b1-a1bd-e93660408c5b"
-          (reference "#PWR019") (unit 1)
-        )
-      )
-    )
-  )
   (symbol (lib_id "Device:C") (at 45.72 68.58 0) (unit 1)
     (in_bom yes) (on_board yes) (dnp no) (fields_autoplaced)
-    (property "Reference" "C11" (at 49.53 67.31 0)
+    (property "Reference" "C15" (at 49.53 67.31 0)
       (effects (font (size 1.27 1.27)) (justify left))
     )
@@
       (project "BLE_REMOTE"
         (path "/3c7105d6-b2e1-4841-966d-0562ae88783f/df7514b4-387c-47b1-a1bd-e93660408c5b"
-          (reference "C11") (unit 1)
+          (reference "C15") (unit 1)
         )
       )
@@
         )
         (path "/3c7105d6-b2e1-4841-966d-0562ae88783f/df7514b4-387c-47b1-a1bd-e93660408c5b"
-          (reference "R12") (unit 1)
+          (reference "R9") (unit 1)
         )
       )
@@
   (symbol (lib_id "power:GND") (at 97.79 166.37 0) (unit 1)
     (in_bom yes) (on_board yes) (dnp no) (fields_autoplaced)
-    (property "Reference" "#PWR040" (at 97.79 172.72 0)
+    (property "Reference" "#PWR018" (at 97.79 172.72 0)
       (effects (font (size 1.27 1.27)) hide)
     )
@@
       (project "BLE_REMOTE"
         (path "/3c7105d6-b2e1-4841-966d-0562ae88783f/df7514b4-387c-47b1-a1bd-e93660408c5b"
-          (reference "#PWR040") (unit 1)
+          (reference "#PWR018") (unit 1)
         )
       )
@@
   (symbol (lib_id "Device:C") (at 176.53 67.31 0) (unit 1)
     (in_bom yes) (on_board yes) (dnp no)
-    (property "Reference" "C13" (at 168.91 66.04 0)
+    (property "Reference" "C17" (at 168.91 66.04 0)
       (effects (font (size 1.27 1.27)) (justify left))
     )
@@
       (project "BLE_REMOTE"
         (path "/3c7105d6-b2e1-4841-966d-0562ae88783f/df7514b4-387c-47b1-a1bd-e93660408c5b"
-          (reference "C13") (unit 1)
+          (reference "C17") (unit 1)
         )
       )
@@
   (symbol (lib_id "power:GND") (at 41.91 118.11 0) (unit 1)
     (in_bom yes) (on_board yes) (dnp no) (fields_autoplaced)
-    (property "Reference" "#PWR012" (at 41.91 124.46 0)
+    (property "Reference" "#PWR013" (at 41.91 124.46 0)
       (effects (font (size 1.27 1.27)) hide)
     )
@@
       (project "BLE_REMOTE"
         (path "/3c7105d6-b2e1-4841-966d-0562ae88783f/df7514b4-387c-47b1-a1bd-e93660408c5b"
-          (reference "#PWR012") (unit 1)
+          (reference "#PWR013") (unit 1)
         )
       )
@@
   (symbol (lib_id "power:GND") (at 45.72 72.39 0) (unit 1)
     (in_bom yes) (on_board yes) (dnp no) (fields_autoplaced)
-    (property "Reference" "#PWR014" (at 45.72 78.74 0)
+    (property "Reference" "#PWR015" (at 45.72 78.74 0)
       (effects (font (size 1.27 1.27)) hide)
     )
@@
       (project "BLE_REMOTE"
         (path "/3c7105d6-b2e1-4841-966d-0562ae88783f/df7514b4-387c-47b1-a1bd-e93660408c5b"
-          (reference "#PWR014") (unit 1)
+          (reference "#PWR015") (unit 1)
         )
       )
@@
   (symbol (lib_id "Connector:Conn_01x03_Pin") (at 102.87 163.83 180) (unit 1)
     (in_bom yes) (on_board yes) (dnp no) (fields_autoplaced)
-    (property "Reference" "J6" (at 104.14 162.56 0)
+    (property "Reference" "J3" (at 104.14 162.56 0)
       (effects (font (size 1.27 1.27)) (justify right))
     )
@@
       (project "BLE_REMOTE"
         (path "/3c7105d6-b2e1-4841-966d-0562ae88783f/df7514b4-387c-47b1-a1bd-e93660408c5b"
-          (reference "J6") (unit 1)
+          (reference "J3") (unit 1)
         )
       )
@@
         )
         (path "/3c7105d6-b2e1-4841-966d-0562ae88783f/df7514b4-387c-47b1-a1bd-e93660408c5b"
-          (reference "R11") (unit 1)
+          (reference "R8") (unit 1)
         )
       )
@@
   (symbol (lib_id "Device:C") (at 226.06 67.31 0) (unit 1)
     (in_bom yes) (on_board yes) (dnp no) (fields_autoplaced)
-    (property "Reference" "C14" (at 229.87 66.04 0)
+    (property "Reference" "C18" (at 229.87 66.04 0)
       (effects (font (size 1.27 1.27)) (justify left))
     )
@@
       (project "BLE_REMOTE"
         (path "/3c7105d6-b2e1-4841-966d-0562ae88783f/df7514b4-387c-47b1-a1bd-e93660408c5b"
-          (reference "C14") (unit 1)
+          (reference "C18") (unit 1)
         )
       )
@@
   (symbol (lib_id "power:VCC") (at 115.57 57.15 0) (unit 1)
     (in_bom yes) (on_board yes) (dnp no) (fields_autoplaced)
-    (property "Reference" "#PWR018" (at 115.57 60.96 0)
+    (property "Reference" "#PWR019" (at 115.57 60.96 0)
       (effects (font (size 1.27 1.27)) hide)
     )
@@
       (project "BLE_REMOTE"
         (path "/3c7105d6-b2e1-4841-966d-0562ae88783f/df7514b4-387c-47b1-a1bd-e93660408c5b"
-          (reference "#PWR018") (unit 1)
+          (reference "#PWR019") (unit 1)
         )
       )
@@
   (symbol (lib_id "power:VCC") (at 59.69 72.39 0) (unit 1)
     (in_bom yes) (on_board yes) (dnp no) (fields_autoplaced)
-    (property "Reference" "#PWR015" (at 59.69 76.2 0)
+    (property "Reference" "#PWR016" (at 59.69 76.2 0)
       (effects (font (size 1.27 1.27)) hide)
     )
@@
       (project "BLE_REMOTE"
         (path "/3c7105d6-b2e1-4841-966d-0562ae88783f/df7514b4-387c-47b1-a1bd-e93660408c5b"
-          (reference "#PWR015") (unit 1)
-        )
-      )
+          (reference "#PWR016") (unit 1)
+        )
+      )
