File: _Electrical/BLE_REMOTE/BLEC_power.kicad_sch (KiCad schematic)
At the start: 19 parts, among them J3 LED, U2 BQ24232RGTR, U3 MIC5528-3.3YMX-TR

Commit message: asdasat
Parts:
- C15: LCSC Part # (none) -> C28323
- C16: LCSC Part # (none) -> C1779
- C17, C18: LCSC Part # (none) -> C23630
- J3: value LED -> LED_STRIP; now left out of the parts list
- R1: LCSC Part # (none) -> C273724
- R10: LCSC Part # (none) -> C25744
- R2, R3, R4, R5, R6: LCSC Part # (none) -> C17168
- R6: LCSC Part # (none) -> C4109
- R7: LCSC Part # (none) -> C334698
- U2: LCSC Part # (none) -> C528622
- U3: value MIC5528-3.3YMX-TR -> MIC5528-3.3YMT-TR; footprint XTDFN6_1P2X1P2_MCH -> _Parts:TDFN6_1P2X1P2_MCH; symbol MIC5528:MIC5528-3.3YMX-TR -> MIC5528_3_3yMT_TR:MIC5528-3.3YMT-TR; LCSC Part # (none) -> C622490
Changed lines of the file:
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@@
   (junction (at 181.61 73.66) (diameter 0) (color 0 0 0 0)
   )
+  (junction (at 233.68 63.5) (diameter 0) (color 0 0 0 0)
+  )
   (junction (at 143.51 62.23) (diameter 0) (color 0 0 0 0)
   )
@@
     (stroke (width 0) (type default))
   )
+  (wire (pts (xy 233.68 63.5) (xy 237.49 63.5))
+    (stroke (width 0) (type default))
+  )
   (wire (pts (xy 222.25 53.34) (xy 242.57 53.34))
     (stroke (width 0) (type default))
@@
     (stroke (width 0) (type default))
   )
-  (wire (pts (xy 226.06 63.5) (xy 237.49 63.5))
+  (wire (pts (xy 226.06 63.5) (xy 233.68 63.5))
     (stroke (width 0) (type default))
   )
@@
       (effects (font (size 1.27 1.27)) hide)
     )
-    (property "LCSC Part #" "" (at 64.77 114.3 0)
+    (property "LCSC Part #" "C334698" (at 64.77 114.3 0)
+      (effects (font (size 1.27 1.27)) hide)
+    )
+    (property "Description" "Extended" (at 64.77 114.3 0)
       (effects (font (size 1.27 1.27)) hide)
     )
@@
       (effects (font (size 1.27 1.27)) hide)
     )
-    (property "LCSC Part #" "" (at 59.69 109.22 0)
+    (property "LCSC Part #" "C17168" (at 59.69 109.22 0)
       (effects (font (size 1.27 1.27)) hide)
     )
@@
       (effects (font (size 1.27 1.27)) hide)
     )
-    (property "LCSC Part #" "" (at 143.51 66.04 0)
+    (property "LCSC Part #" "C1779" (at 143.51 66.04 0)
       (effects (font (size 1.27 1.27)) hide)
     )
@@
       (effects (font (size 1.27 1.27)) hide)
     )
-    (property "LCSC Part #" "" (at 45.72 68.58 0)
+    (property "LCSC Part #" "C28323" (at 45.72 68.58 0)
       (effects (font (size 1.27 1.27)) hide)
     )
@@
       (effects (font (size 1.27 1.27)) hide)
     )
-    (property "LCSC Part #" "" (at 54.61 104.14 0)
+    (property "LCSC Part #" "C17168" (at 54.61 104.14 0)
       (effects (font (size 1.27 1.27)) hide)
     )
@@
       (effects (font (size 1.27 1.27)) hide)
     )
-    (property "LCSC Part #" "" (at 134.62 69.85 0)
+    (property "LCSC Part #" "C4109" (at 134.62 69.85 0)
       (effects (font (size 1.27 1.27)) hide)
     )
@@
     )
   )
-  (symbol (lib_id "MIC5528:MIC5528-3.3YMX-TR") (at 222.25 64.77 180) (unit 1)
+  (symbol (lib_id "MIC5528_3_3yMT_TR:MIC5528-3.3YMT-TR") (at 222.25 64.77 180) (unit 1)
     (in_bom yes) (on_board yes) (dnp no) (fields_autoplaced)
     (property "Reference" "U3" (at 201.93 46.99 0)
       (effects (font (size 1.524 1.524)))
     )
-    (property "Value" "MIC5528-3.3YMX-TR" (at 201.93 49.53 0)
+    (property "Value" "MIC5528-3.3YMT-TR" (at 201.93 72.39 0)
       (effects (font (size 1.524 1.524)))
     )
-    (property "Footprint" "XTDFN6_1P2X1P2_MCH" (at 222.25 67.31 0)
+    (property "Footprint" "_Parts:TDFN6_1P2X1P2_MCH" (at 222.25 64.77 0)
       (effects (font (size 1.27 1.27) italic) hide)
     )
-    (property "Datasheet" "https://www.digikey.ca/en/products/detail/microchip-technology/MIC5528-3-3YMT-TR/4864020" (at 222.25 66.04 0)
+    (property "Datasheet" "MIC5528-3.3YMT-TR" (at 222.25 64.77 0)
       (effects (font (size 1.27 1.27) italic) hide)
     )
@@
       (effects (font (size 1.27 1.27)) hide)
     )
-    (property "LCSC Part #" "" (at 222.25 64.77 0)
-      (effects (font (size 1.27 1.27)) hide)
-    )
+    (property "LCSC Part #" "C622490" (at 222.25 64.77 0)
+      (effects (font (size 1.27 1.27)) hide)
+    )
+    (property "Description" "Extended" (at 222.25 64.77 0)
+      (effects (font (size 1.27 1.27)) hide)
+    )
+    (pin "1")
+    (pin "2")
     (pin "3")
     (pin "4")
     (pin "5")
     (pin "6")
-    (pin "1")
-    (pin "2")
     (pin "7")
     (instances
@@
         (path "/3c7105d6-b2e1-4841-966d-0562ae88783f/df7514b4-387c-47b1-a1bd-e93660408c5b"
           (reference "U3") (unit 1)
+        )
+      )
+    )
+  )
+  (symbol (lib_id "power:PWR_FLAG") (at 233.68 63.5 0) (unit 1)
+    (in_bom yes) (on_board yes) (dnp no) (fields_autoplaced)
+    (property "Reference" "#FLG06" (at 233.68 61.595 0)
+      (effects (font (size 1.27 1.27)) hide)
+    )
+    (property "Value" "PWR_FLAG" (at 233.68 59.69 0)
+      (effects (font (size 1.27 1.27)))
+    )
+    (property "Footprint" "" (at 233.68 63.5 0)
+      (effects (font (size 1.27 1.27)) hide)
+    )
+    (property "Datasheet" "~" (at 233.68 63.5 0)
+      (effects (font (size 1.27 1.27)) hide)
+    )
+    (pin "1")
+    (instances
+      (project "BLE_REMOTE"
+        (path "/3c7105d6-b2e1-4841-966d-0562ae88783f/df7514b4-387c-47b1-a1bd-e93660408c5b"
+          (reference "#FLG06") (unit 1)
         )
       )
@@
       (effects (font (size 1.27 1.27)) hide)
     )
-    (property "LCSC Part #" "" (at 176.53 67.31 0)
+    (property "LCSC Part #" "C23630" (at 176.53 67.31 0)
       (effects (font (size 1.27 1.27)) hide)
     )
@@
       (effects (font (size 1.27 1.27)) hide)
     )
-    (property "LCSC Part #" "" (at 135.89 100.33 0)
+    (property "LCSC Part #" "C25744" (at 135.89 100.33 0)
       (effects (font (size 1.27 1.27)) hide)
     )
@@
   )
   (symbol (lib_id "Connector:Conn_01x03_Pin") (at 102.87 163.83 180) (unit 1)
-    (in_bom yes) (on_board yes) (dnp no) (fields_autoplaced)
+    (in_bom no) (on_board yes) (dnp no) (fields_autoplaced)
     (property "Reference" "J3" (at 104.14 162.56 0)
       (effects (font (size 1.27 1.27)) (justify right))
     )
-    (property "Value" "LED" (at 104.14 165.1 0)
+    (property "Value" "LED_STRIP" (at 104.14 165.1 0)
       (effects (font (size 1.27 1.27)) (justify right))
     )
@@
       (effects (font (size 1.27 1.27)) hide)
     )
-    (property "LCSC Part #" "" (at 45.72 91.44 0)
+    (property "LCSC Part #" "C17168" (at 45.72 91.44 0)
       (effects (font (size 1.27 1.27)) hide)
     )
@@
       (effects (font (size 1.27 1.27)) hide)
     )
-    (property "LCSC Part #" "" (at 41.91 86.36 0)
+    (property "LCSC Part #" "C273724" (at 41.91 86.36 0)
+      (effects (font (size 1.27 1.27)) hide)
+    )
+    (property "Description" "Extended" (at 41.91 86.36 0)
       (effects (font (size 1.27 1.27)) hide)
     )
@@
       (effects (font (size 1.27 1.27)) hide)
     )
-    (property "LCSC Part #" "" (at 123.19 69.85 0)
+    (property "LCSC Part #" "C4109" (at 123.19 69.85 0)
       (effects (font (size 1.27 1.27)) hide)
     )
@@
       (effects (font (size 1.27 1.27)) hide)
     )
-    (property "LCSC Part #" "" (at 95.25 92.71 0)
+    (property "LCSC Part #" "C528622" (at 95.25 92.71 0)
+      (effects (font (size 1.27 1.27)) hide)
+    )
+    (property "Description" "Extended" (at 95.25 92.71 0)
       (effects (font (size 1.27 1.27)) hide)
     )
@@
       (effects (font (size 1.27 1.27)) hide)
     )
-    (property "LCSC Part #" "" (at 226.06 67.31 0)
+    (property "LCSC Part #" "C23630" (at 226.06 67.31 0)
       (effects (font (size 1.27 1.27)) hide)
     )
@@
       (effects (font (size 1.27 1.27)) hide)
     )
-    (property "LCSC Part #" "" (at 49.53 99.06 0)
+    (property "LCSC Part #" "C17168" (at 49.53 99.06 0)
       (effects (font (size 1.27 1.27)) hide)
     )
@@
       (effects (font (size 1.27 1.27)) hide)
     )
-    (property "LCSC Part #" "" (at 59.69 76.2 0)
-      (effects (font (size 1.27 1.27)) hide)
-    )
+    (property "LCSC Part #" "C17168" (at 59.69 76.2 0)
+      (effects (font (size 1.27 1.27)) hide)
+    )
