File: _Electrical/BLE_REMOTE/BLE_C_MCU.kicad_sch (KiCad schematic)
At the start: 16 parts, among them J1 PGRM, J2 Conn_01x02_Pin, U1 nRF52832-QFxx, Y1 Crystal_GND24

Commit message: JLCPCB parts selected
Parts:
- L1: LCSC Part # (none) -> C412343
- Y1: JLCPCB Part# (none) -> C1985928; LCSC Part # (none) -> C7294588
Connections:
- no-connect marks 20 -> 21
Changed lines of the file:
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@@
   (no_connect (at 137.16 120.65))
   (no_connect (at 137.16 74.93))
+  (no_connect (at 137.16 85.09))
   (wire (pts (xy 36.83 107.95) (xy 36.83 118.11))
     (stroke (width 0) (type default))
@@
       (effects (font (size 1.27 1.27)) hide)
     )
+    (property "JLCPCB Part#" "C1985928" (at 50.8 102.87 0)
+      (effects (font (size 1.27 1.27)) hide)
+    )
+    (property "LCSC Part #" "C7294588" (at 50.8 102.87 0)
+      (effects (font (size 1.27 1.27)) hide)
+    )
     (pin "1")
     (pin "2")
@@
       (effects (font (size 1.27 1.27)) hide)
     )
+    (property "JLCPCB Part#" "" (at 104.14 44.45 0)
+      (effects (font (size 1.27 1.27)) hide)
+    )
+    (property "LCSC Part #" "" (at 104.14 44.45 0)
+      (effects (font (size 1.27 1.27)) hide)
+    )
     (pin "1")
     (pin "2")
@@
       (effects (font (size 1.27 1.27)) hide)
     )
+    (property "JLCPCB Part#" "" (at 147.32 50.8 0)
+      (effects (font (size 1.27 1.27)) hide)
+    )
+    (property "LCSC Part #" "" (at 147.32 50.8 0)
+      (effects (font (size 1.27 1.27)) hide)
+    )
     (pin "1")
     (pin "2")
@@
     )
     (property "Part" "GJM1555C1H100FB01D" (at 43.18 107.95 0)
+      (effects (font (size 1.27 1.27)) hide)
+    )
+    (property "JLCPCB Part#" "" (at 43.18 107.95 0)
+      (effects (font (size 1.27 1.27)) hide)
+    )
+    (property "LCSC Part #" "" (at 43.18 107.95 0)
       (effects (font (size 1.27 1.27)) hide)
     )
@@
       (effects (font (size 1.27 1.27)) hide)
     )
+    (property "JLCPCB Part#" "" (at 99.06 44.45 0)
+      (effects (font (size 1.27 1.27)) hide)
+    )
+    (property "LCSC Part #" "" (at 99.06 44.45 0)
+      (effects (font (size 1.27 1.27)) hide)
+    )
     (pin "1")
     (pin "2")
@@
       (effects (font (size 1.27 1.27)) hide)
     )
+    (property "JLCPCB Part#" "" (at 147.32 55.88 0)
+      (effects (font (size 1.27 1.27)) hide)
+    )
+    (property "LCSC Part #" "" (at 147.32 55.88 0)
+      (effects (font (size 1.27 1.27)) hide)
+    )
     (pin "1")
     (pin "2")
@@
       (effects (font (size 1.524 1.524)) hide)
     )
+    (property "JLCPCB Part#" "" (at 48.26 69.85 0)
+      (effects (font (size 1.27 1.27)) hide)
+    )
+    (property "LCSC Part #" "" (at 48.26 69.85 0)
+      (effects (font (size 1.27 1.27)) hide)
+    )
+    (pin "1")
+    (pin "2")
     (pin "4")
     (pin "5")
-    (pin "1")
-    (pin "2")
     (instances
       (project "BLE_REMOTE"
@@
       (effects (font (size 1.27 1.27)) hide)
     )
+    (property "JLCPCB Part#" "" (at 76.2 118.11 0)
+      (effects (font (size 1.27 1.27)) hide)
+    )
+    (property "LCSC Part #" "" (at 76.2 118.11 0)
+      (effects (font (size 1.27 1.27)) hide)
+    )
     (pin "1")
     (pin "2")
@@
       (effects (font (size 1.27 1.27)) hide)
     )
+    (property "JLCPCB Part#" "" (at 58.42 138.43 0)
+      (effects (font (size 1.27 1.27)) hide)
+    )
+    (property "LCSC Part #" "" (at 58.42 138.43 0)
+      (effects (font (size 1.27 1.27)) hide)
+    )
     (pin "1")
     (pin "2")
@@
     )
     (property "Part" "GJM1555C1HR80BB01D" (at 78.74 88.9 0)
+      (effects (font (size 1.27 1.27)) hide)
+    )
+    (property "JLCPCB Part#" "" (at 78.74 88.9 0)
+      (effects (font (size 1.27 1.27)) hide)
+    )
+    (property "LCSC Part #" "" (at 78.74 88.9 0)
       (effects (font (size 1.27 1.27)) hide)
     )
@@
       (effects (font (size 1.27 1.27)) hide)
     )
+    (property "JLCPCB Part#" "" (at 114.3 44.45 0)
+      (effects (font (size 1.27 1.27)) hide)
+    )
+    (property "LCSC Part #" "" (at 114.3 44.45 0)
+      (effects (font (size 1.27 1.27)) hide)
+    )
     (pin "1")
     (pin "2")
@@
     )
     (property "Part" "NRF52832-QFAA-R" (at 114.3 102.87 0)
+      (effects (font (size 1.27 1.27)) hide)
+    )
+    (property "JLCPCB Part#" "" (at 114.3 102.87 0)
+      (effects (font (size 1.27 1.27)) hide)
+    )
+    (property "LCSC Part #" "" (at 114.3 102.87 0)
       (effects (font (size 1.27 1.27)) hide)
     )
@@
       (effects (font (size 1.27 1.27)) hide)
     )
+    (property "JLCPCB Part#" "" (at 41.91 97.79 0)
+      (effects (font (size 1.27 1.27)) hide)
+    )
+    (property "LCSC Part #" "" (at 41.91 97.79 0)
+      (effects (font (size 1.27 1.27)) hide)
+    )
     (pin "1")
     (pin "2")
@@
     )
     (property "Part" "LQW15AN3N9G80D" (at 71.12 85.09 90)
+      (effects (font (size 1.27 1.27)) hide)
+    )
+    (property "JLCPCB Part#" "" (at 71.12 85.09 0)
+      (effects (font (size 1.27 1.27)) hide)
+    )
+    (property "LCSC Part #" "C412343" (at 71.12 85.09 0)
       (effects (font (size 1.27 1.27)) hide)
     )
@@
       (effects (font (size 1.27 1.27)) hide)
     )
+    (property "JLCPCB Part#" "" (at 147.32 45.72 0)
+      (effects (font (size 1.27 1.27)) hide)
+    )
+    (property "LCSC Part #" "" (at 147.32 45.72 0)
+      (effects (font (size 1.27 1.27)) hide)
+    )
     (pin "1")
     (pin "2")
@@
       (effects (font (size 1.27 1.27)) hide)
     )
+    (property "JLCPCB Part#" "" (at 109.22 44.45 0)
+      (effects (font (size 1.27 1.27)) hide)
+    )
+    (property "LCSC Part #" "" (at 109.22 44.45 0)
+      (effects (font (size 1.27 1.27)) hide)
+    )

Commit message: Adjusted components and changed buttons
Parts:
- Y1: JLCPCB Part# C1985928 -> C2901738; LCSC Part # C7294588 -> C2901738
- renumbered C6 to C10, C7 to C11, C8 to C12, C9 to C13, C10 to C14, C1 to C5, C2 to C6, C3 to C7, C4 to C8, C5 to C9
