File: _Electrical/BLE_REMOTE/BLE_C_MCU.kicad_sch (KiCad schematic)
At the start: 16 parts, among them J1 PGRM, J2 Conn_01x02_Pin, U1 nRF52832-QFxx, Y1 Crystal_GND24

Commit message: asdasat
Parts:
- C10: LCSC Part # (none) -> C1546
- C11: LCSC Part # (none) -> C15849
- C12, C14, C8: LCSC Part # (none) -> C1525
- C13: LCSC Part # (none) -> C1779
- C5, C6: LCSC Part # (none) -> C32949
- C7: LCSC Part # (none) -> C327032
- J1: now left out of the parts list
- J2: value Conn_01x02_Pin -> RESET; now left out of the parts list
- U1: LCSC Part # (none) -> C77540
Changed lines of the file:
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@@
       (effects (font (size 1.27 1.27)) hide)
     )
-    (property "LCSC Part #" "" (at 147.32 50.8 0)
+    (property "LCSC Part #" "C1779" (at 147.32 50.8 0)
       (effects (font (size 1.27 1.27)) hide)
     )
@@
       (effects (font (size 1.27 1.27)) hide)
     )
-    (property "LCSC Part #" "" (at 43.18 107.95 0)
+    (property "LCSC Part #" "C32949" (at 43.18 107.95 0)
       (effects (font (size 1.27 1.27)) hide)
     )
@@
       (effects (font (size 1.27 1.27)) hide)
     )
+    (property "Description" "Extended" (at 50.8 102.87 0)
+      (effects (font (size 1.27 1.27)) hide)
+    )
     (pin "1")
     (pin "2")
@@
       (effects (font (size 1.27 1.27)) hide)
     )
-    (property "LCSC Part #" "" (at 99.06 44.45 0)
+    (property "LCSC Part #" "C1525" (at 99.06 44.45 0)
       (effects (font (size 1.27 1.27)) hide)
     )
@@
       (effects (font (size 1.27 1.27)) hide)
     )
-    (property "LCSC Part #" "" (at 147.32 55.88 0)
+    (property "LCSC Part #" "C1525" (at 147.32 55.88 0)
       (effects (font (size 1.27 1.27)) hide)
     )
@@
   )
   (symbol (lib_id "Connector:Conn_01x02_Pin") (at 76.2 118.11 0) (unit 1)
-    (in_bom yes) (on_board yes) (dnp no)
+    (in_bom no) (on_board yes) (dnp no)
     (property "Reference" "J2" (at 73.66 119.38 0)
       (effects (font (size 1.27 1.27)))
     )
-    (property "Value" "Conn_01x02_Pin" (at 55.88 128.27 0)
+    (property "Value" "RESET" (at 55.88 128.27 0)
       (effects (font (size 1.27 1.27)) hide)
     )
@@
   )
   (symbol (lib_id "Connector_Generic:Conn_01x04") (at 58.42 138.43 180) (unit 1)
-    (in_bom yes) (on_board yes) (dnp no)
+    (in_bom no) (on_board yes) (dnp no)
     (property "Reference" "J1" (at 54.61 138.43 0)
       (effects (font (size 1.27 1.27)))
@@
       (effects (font (size 1.27 1.27)) hide)
     )
-    (property "LCSC Part #" "" (at 78.74 88.9 0)
+    (property "LCSC Part #" "C327032" (at 78.74 88.9 0)
+      (effects (font (size 1.27 1.27)) hide)
+    )
+    (property "Description" "Extended" (at 78.74 88.9 0)
       (effects (font (size 1.27 1.27)) hide)
     )
@@
       (effects (font (size 1.27 1.27)) hide)
     )
-    (property "LCSC Part #" "" (at 114.3 44.45 0)
+    (property "LCSC Part #" "C15849" (at 114.3 44.45 0)
       (effects (font (size 1.27 1.27)) hide)
     )
@@
       (effects (font (size 1.27 1.27)) hide)
     )
-    (property "LCSC Part #" "" (at 114.3 102.87 0)
+    (property "LCSC Part #" "C77540" (at 114.3 102.87 0)
+      (effects (font (size 1.27 1.27)) hide)
+    )
+    (property "Description" "Extended" (at 114.3 102.87 0)
       (effects (font (size 1.27 1.27)) hide)
     )
@@
       (effects (font (size 1.27 1.27)) hide)
     )
-    (property "LCSC Part #" "" (at 41.91 97.79 0)
+    (property "LCSC Part #" "C32949" (at 41.91 97.79 0)
       (effects (font (size 1.27 1.27)) hide)
     )
@@
     )
     (property "LCSC Part #" "C412343" (at 71.12 85.09 0)
+      (effects (font (size 1.27 1.27)) hide)
+    )
+    (property "Description" "Extended" (at 71.12 85.09 0)
       (effects (font (size 1.27 1.27)) hide)
     )
@@
       (effects (font (size 1.27 1.27)) hide)
     )
-    (property "LCSC Part #" "" (at 147.32 45.72 0)
+    (property "LCSC Part #" "C1525" (at 147.32 45.72 0)
       (effects (font (size 1.27 1.27)) hide)
     )
@@
       (effects (font (size 1.27 1.27)) hide)
     )
-    (property "LCSC Part #" "" (at 109.22 44.45 0)
-      (effects (font (size 1.27 1.27)) hide)
-    )
+    (property "LCSC Part #" "C1546" (at 109.22 44.45 0)
+      (effects (font (size 1.27 1.27)) hide)
+    )

Commit message: ordered from JLCPCB
Parts:
- J2: footprint Connector_PinHeader_1.27mm:PinHeader_1x02_P1.27mm_Vertical -> Connector_PinHeader_1.27mm:PinHeader_2x01_P1.27mm_Vertical_SMD
Changed lines of the file:
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@@
       (effects (font (size 1.27 1.27)) hide)
     )
-    (property "Footprint" "Connector_PinHeader_1.27mm:PinHeader_1x02_P1.27mm_Vertical" (at 76.2 118.11 0)
+    (property "Footprint" "Connector_PinHeader_1.27mm:PinHeader_2x01_P1.27mm_Vertical_SMD" (at 76.2 118.11 0)
       (effects (font (size 1.27 1.27)) hide)
     )
