File: _Electrical/BLE_REMOTE/BLEC_peripherals.kicad_sch (KiCad schematic)
At the start: 17 parts, among them J4 BUZZER, J4 SWITCH, J6 Display, Q1 BSS806NEH6327XTSA1, Q2 NPN, SW1 SW_Push

Commit message: asdasat
Parts:
- C17: LCSC Part # (none) -> C1779
- C19: LCSC Part # (none) -> C1523
- J4, J6: now left out of the parts list
- J4: LCSC Part # (none) -> C2759981
- L2: LCSC Part # (none) -> C1046
- R11, R12: LCSC Part # (none) -> C4109
- R13: LCSC Part # (none) -> C25091
- R14, R15, R16: LCSC Part # (none) -> C25792
Connections:
- net BUTTON: now also SW1.2
- net GND: now also SW1.3
- no-connect marks 2 -> 0
Changed lines of the file:
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@@
   (junction (at 171.45 93.98) (diameter 0) (color 0 0 0 0)
   )
+  (junction (at 45.72 73.66) (diameter 0) (color 0 0 0 0)
+  )
   (junction (at 148.59 44.45) (diameter 0) (color 0 0 0 0)
   )
@@
   (junction (at 99.06 73.66) (diameter 0) (color 0 0 0 0)
   )
-  (no_connect (at 71.12 73.66))
-  (no_connect (at 45.72 83.82))
   (wire (pts (xy 34.29 40.64) (xy 39.37 40.64))
     (stroke (width 0) (type default))
@@
     (stroke (width 0) (type default))
   )
+  (wire (pts (xy 71.12 73.66) (xy 71.12 62.23))
+    (stroke (width 0) (type default))
+  )
   (wire (pts (xy 69.85 100.33) (xy 69.85 105.41))
     (stroke (width 0) (type default))
@@
     (stroke (width 0) (type default))
   )
+  (wire (pts (xy 71.12 62.23) (xy 45.72 62.23))
+    (stroke (width 0) (type default))
+  )
   (wire (pts (xy 148.59 31.75) (xy 148.59 44.45))
     (stroke (width 0) (type default))
@@
   )
   (wire (pts (xy 69.85 105.41) (xy 71.12 105.41))
+    (stroke (width 0) (type default))
+  )
+  (wire (pts (xy 45.72 62.23) (xy 45.72 73.66))
     (stroke (width 0) (type default))
   )
@@
       (effects (font (size 1.27 1.27)) hide)
     )
-    (property "LCSC Part #" "" (at 121.92 31.75 0)
+    (property "LCSC Part #" "C1046" (at 121.92 31.75 0)
       (effects (font (size 1.27 1.27)) hide)
     )
@@
       (effects (font (size 1.27 1.27)) hide)
     )
-    (property "LCSC Part #" "" (at 104.14 60.96 0)
+    (property "LCSC Part #" "C25091" (at 104.14 60.96 0)
       (effects (font (size 1.27 1.27)) hide)
     )
@@
       (effects (font (size 1.27 1.27)) hide)
     )
-    (property "LCSC Part #" "" (at 138.43 48.26 0)
+    (property "LCSC Part #" "C1779" (at 138.43 48.26 0)
       (effects (font (size 1.27 1.27)) hide)
     )
@@
   )
   (symbol (lib_id "Connector:Conn_01x02_Pin") (at 76.2 107.95 180) (unit 1)
-    (in_bom yes) (on_board yes) (dnp no)
+    (in_bom no) (on_board yes) (dnp no)
     (property "Reference" "J4" (at 77.47 105.41 0)
       (effects (font (size 1.27 1.27)) (justify right))
@@
       (effects (font (size 1.27 1.27)) (justify bottom) hide)
     )
-    (property "Description" "\nTS-1187A-B-A-B XKB Connectivity\n" (at 58.42 78.74 0)
+    (property "Description" "Digikey" (at 58.42 78.74 0)
       (effects (font (size 1.27 1.27)) (justify bottom) hide)
     )
@@
       (effects (font (size 1.27 1.27)) hide)
     )
+    (pin "1")
+    (pin "2")
+    (pin "3")
     (pin "4")
-    (pin "1")
-    (pin "2")
-    (pin "3")
     (instances
       (project "BLE_REMOTE"
@@
       (effects (font (size 1.27 1.27)) hide)
     )
-    (property "LCSC Part #" "" (at 171.45 97.79 0)
+    (property "LCSC Part #" "C25792" (at 171.45 97.79 0)
       (effects (font (size 1.27 1.27)) hide)
     )
@@
       (effects (font (size 1.27 1.27)) hide)
     )
-    (property "LCSC Part #" "" (at 50.8 54.61 0)
+    (property "LCSC Part #" "C4109" (at 50.8 54.61 0)
       (effects (font (size 1.27 1.27)) hide)
     )
@@
       (effects (font (size 1.27 1.27)) hide)
     )
-    (property "LCSC Part #" "" (at 161.29 97.79 0)
+    (property "LCSC Part #" "C25792" (at 161.29 97.79 0)
       (effects (font (size 1.27 1.27)) hide)
     )
@@
         (path "/3c7105d6-b2e1-4841-966d-0562ae88783f/3c7d46da-db2c-458d-86d8-33d657630bb5"
           (reference "R17") (unit 1)
+        )
+      )
+    )
+  )
+  (symbol (lib_id "power:GND") (at 45.72 83.82 0) (unit 1)
+    (in_bom yes) (on_board yes) (dnp no) (fields_autoplaced)
+    (property "Reference" "#PWR043" (at 45.72 90.17 0)
+      (effects (font (size 1.27 1.27)) hide)
+    )
+    (property "Value" "GND" (at 45.72 88.9 0)
+      (effects (font (size 1.27 1.27)))
+    )
+    (property "Footprint" "" (at 45.72 83.82 0)
+      (effects (font (size 1.27 1.27)) hide)
+    )
+    (property "Datasheet" "" (at 45.72 83.82 0)
+      (effects (font (size 1.27 1.27)) hide)
+    )
+    (pin "1")
+    (instances
+      (project "BLE_REMOTE"
+        (path "/3c7105d6-b2e1-4841-966d-0562ae88783f/01d40fd6-ccdc-442b-bfe3-30d4d8ca438d"
+          (reference "#PWR043") (unit 1)
         )
       )
@@
       (effects (font (size 1.27 1.27)) hide)
     )
-    (property "LCSC Part #" "" (at 153.67 48.26 0)
+    (property "LCSC Part #" "C2759981" (at 153.67 48.26 0)
+      (effects (font (size 1.27 1.27)) hide)
+    )
+    (property "Description" "Extended" (at 153.67 48.26 0)
       (effects (font (size 1.27 1.27)) hide)
     )
@@
       (effects (font (size 1.27 1.27)) hide)
     )
-    (property "LCSC Part #" "" (at 50.8 40.64 0)
+    (property "LCSC Part #" "C4109" (at 50.8 40.64 0)
       (effects (font (size 1.27 1.27)) hide)
     )
@@
   )
   (symbol (lib_id "Connector_Generic:Conn_01x04") (at 170.18 111.76 0) (unit 1)
-    (in_bom yes) (on_board yes) (dnp no)
+    (in_bom no) (on_board yes) (dnp no)
     (property "Reference" "J6" (at 172.72 111.76 0)
       (effects (font (size 1.27 1.27)) (justify left))
@@
       (effects (font (size 1.27 1.27)) hide)
     )
-    (property "LCSC Part #" "" (at 127 35.56 0)
+    (property "LCSC Part #" "C1523" (at 127 35.56 0)
       (effects (font (size 1.27 1.27)) hide)
     )
@@
       (effects (font (size 1.27 1.27)) hide)
     )
-    (property "LCSC Part #" "" (at 114.3 77.47 0)
-      (effects (font (size 1.27 1.27)) hide)
-    )
+    (property "LCSC Part #" "C25792" (at 114.3 77.47 0)
+      (effects (font (size 1.27 1.27)) hide)
+    )

Commit message: ordered from JLCPCB
Parts:
- added C15 (x2): 10uF, Capacitor_SMD:C_0402_1005Metric_Pad0.74x0.62mm_HandSolder, symbol Device:C
- added R32, R33: 2k, Resistor_SMD:R_0402_1005Metric_Pad0.72x0.64mm_HandSolder, symbol Device:R
Connections:
- net BUTTON: now also C15.2, R33.2; no longer SW1.1, SW1.2
- net GND: now also C15.1, C15.1
- net SWITCH: now also C15.2, R32.2; no longer J4.2 (Pin_2)
- new net: J4.2 (Pin_2), R32.1
- new net: R33.1, SW1.1, SW1.2
