File: _Electrical/BLE_REMOTE/BLE_REMOTE.kicad_sch (KiCad schematic)
At the start: 8 parts

Commit message: ordered from JLCPCB
Parts:
- removed R25 (x4): 0R, Resistor_SMD:R_0402_1005Metric_Pad0.72x0.64mm_HandSolder, symbol Device:R
Connections:
- net GND: now also H1.1, H2.1, H3.1, H4.1
Changed lines of the file:
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@@
   (junction (at 223.52 143.51) (diameter 0) (color 0 0 0 0)
+  )
+  (junction (at 247.65 143.51) (diameter 0) (color 0 0 0 0)
   )
   (junction (at 199.39 143.51) (diameter 0) (color 0 0 0 0)
   )
-  (junction (at 247.65 143.51) (diameter 0) (color 0 0 0 0)
+  (wire (pts (xy 223.52 133.35) (xy 223.52 143.51))
+    (stroke (width 0) (type default))
   )
   (wire (pts (xy 247.65 143.51) (xy 247.65 153.67))
     (stroke (width 0) (type default))
   )
-  (wire (pts (xy 199.39 135.89) (xy 199.39 133.35))
+  (wire (pts (xy 199.39 133.35) (xy 199.39 143.51))
     (stroke (width 0) (type default))
   )
-  (wire (pts (xy 172.72 143.51) (xy 199.39 143.51))
-    (stroke (width 0) (type default))
-  )
-  (wire (pts (xy 172.72 135.89) (xy 172.72 133.35))
-    (stroke (width 0) (type default))
-  )
-  (wire (pts (xy 247.65 142.24) (xy 247.65 143.51))
-    (stroke (width 0) (type default))
-  )
-  (wire (pts (xy 223.52 133.35) (xy 223.52 135.89))
+  (wire (pts (xy 172.72 133.35) (xy 172.72 143.51))
     (stroke (width 0) (type default))
   )
@@
     (stroke (width 0) (type default))
   )
+  (wire (pts (xy 247.65 134.62) (xy 247.65 143.51))
+    (stroke (width 0) (type default))
+  )
   (wire (pts (xy 199.39 143.51) (xy 223.52 143.51))
+    (stroke (width 0) (type default))
+  )
+  (wire (pts (xy 172.72 143.51) (xy 199.39 143.51))
     (stroke (width 0) (type default))
   )
@@
         (path "/3c7105d6-b2e1-4841-966d-0562ae88783f"
           (reference "H4") (unit 1)
-        )
-      )
-    )
-  )
-  (symbol (lib_id "Device:R") (at 199.39 139.7 0) (unit 1)
-    (in_bom yes) (on_board yes) (dnp no)
-    (property "Reference" "R25" (at 196.85 139.7 90)
-      (effects (font (size 1.27 1.27)))
-    )
-    (property "Value" "0R" (at 199.39 139.7 90)
-      (effects (font (size 1.27 1.27)))
-    )
-    (property "Footprint" "Resistor_SMD:R_0402_1005Metric_Pad0.72x0.64mm_HandSolder" (at 197.612 139.7 90)
-      (effects (font (size 1.27 1.27)) hide)
-    )
-    (property "Datasheet" "https://www.digikey.ca/en/products/detail/yageo/RC0402FR-07100KL/726526" (at 199.39 139.7 0)
-      (effects (font (size 1.27 1.27)) hide)
-    )
-    (property "Part" "RC0402JR-070RL" (at 199.39 139.7 90)
-      (effects (font (size 1.27 1.27)) hide)
-    )
-    (property "JLCPCB Part#" "" (at 199.39 139.7 0)
-      (effects (font (size 1.27 1.27)) hide)
-    )
-    (property "LCSC Part #" "C17168" (at 199.39 139.7 0)
-      (effects (font (size 1.27 1.27)) hide)
-    )
-    (pin "1")
-    (pin "2")
-    (instances
-      (project "BLE_REMOTE"
-        (path "/3c7105d6-b2e1-4841-966d-0562ae88783f/df7514b4-387c-47b1-a1bd-e93660408c5b"
-          (reference "R25") (unit 1)
-        )
-        (path "/3c7105d6-b2e1-4841-966d-0562ae88783f/df7514b4-387c-47b1-a1bd-e93660408c5b/a095a39f-6b3f-4eb2-81ef-a7fa39c10239"
-          (reference "R23") (unit 1)
-        )
-        (path "/3c7105d6-b2e1-4841-966d-0562ae88783f/df7514b4-387c-47b1-a1bd-e93660408c5b/a0a15605-c20d-4158-a513-aa16071bb857"
-          (reference "R27") (unit 1)
-        )
-        (path "/3c7105d6-b2e1-4841-966d-0562ae88783f"
-          (reference "R29") (unit 1)
-        )
-      )
-      (project "Battery"
-        (path "/671d4de1-777a-48e9-9f3d-613423e17047"
-          (reference "R1") (unit 1)
-        )
-      )
-      (project "BLEC_power"
-        (path "/a7925ddf-5c61-458f-8a66-a1453f1c9b4d"
-          (reference "R25") (unit 1)
-        )
-      )
-    )
-  )
-  (symbol (lib_id "Device:R") (at 172.72 139.7 0) (unit 1)
-    (in_bom yes) (on_board yes) (dnp no)
-    (property "Reference" "R25" (at 170.18 139.7 90)
-      (effects (font (size 1.27 1.27)))
-    )
-    (property "Value" "0R" (at 172.72 139.7 90)
-      (effects (font (size 1.27 1.27)))
-    )
-    (property "Footprint" "Resistor_SMD:R_0402_1005Metric_Pad0.72x0.64mm_HandSolder" (at 170.942 139.7 90)
-      (effects (font (size 1.27 1.27)) hide)
-    )
-    (property "Datasheet" "https://www.digikey.ca/en/products/detail/yageo/RC0402FR-07100KL/726526" (at 172.72 139.7 0)
-      (effects (font (size 1.27 1.27)) hide)
-    )
-    (property "Part" "RC0402JR-070RL" (at 172.72 139.7 90)
-      (effects (font (size 1.27 1.27)) hide)
-    )
-    (property "JLCPCB Part#" "" (at 172.72 139.7 0)
-      (effects (font (size 1.27 1.27)) hide)
-    )
-    (property "LCSC Part #" "C17168" (at 172.72 139.7 0)
-      (effects (font (size 1.27 1.27)) hide)
-    )
-    (pin "1")
-    (pin "2")
-    (instances
-      (project "BLE_REMOTE"
-        (path "/3c7105d6-b2e1-4841-966d-0562ae88783f/df7514b4-387c-47b1-a1bd-e93660408c5b"
-          (reference "R25") (unit 1)
-        )
-        (path "/3c7105d6-b2e1-4841-966d-0562ae88783f/df7514b4-387c-47b1-a1bd-e93660408c5b/a095a39f-6b3f-4eb2-81ef-a7fa39c10239"
-          (reference "R23") (unit 1)
-        )
-        (path "/3c7105d6-b2e1-4841-966d-0562ae88783f/df7514b4-387c-47b1-a1bd-e93660408c5b/a0a15605-c20d-4158-a513-aa16071bb857"
-          (reference "R27") (unit 1)
-        )
-        (path "/3c7105d6-b2e1-4841-966d-0562ae88783f"
-          (reference "R28") (unit 1)
-        )
-      )
-      (project "Battery"
-        (path "/671d4de1-777a-48e9-9f3d-613423e17047"
-          (reference "R1") (unit 1)
-        )
-      )
-      (project "BLEC_power"
-        (path "/a7925ddf-5c61-458f-8a66-a1453f1c9b4d"
-          (reference "R25") (unit 1)
-        )
-      )
-    )
-  )
-  (symbol (lib_id "Device:R") (at 247.65 138.43 0) (unit 1)
-    (in_bom yes) (on_board yes) (dnp no)
-    (property "Reference" "R25" (at 245.11 138.43 90)
-      (effects (font (size 1.27 1.27)))
-    )
-    (property "Value" "0R" (at 247.65 138.43 90)
-      (effects (font (size 1.27 1.27)))
-    )
-    (property "Footprint" "Resistor_SMD:R_0402_1005Metric_Pad0.72x0.64mm_HandSolder" (at 245.872 138.43 90)
-      (effects (font (size 1.27 1.27)) hide)
-    )
-    (property "Datasheet" "https://www.digikey.ca/en/products/detail/yageo/RC0402FR-07100KL/726526" (at 247.65 138.43 0)
-      (effects (font (size 1.27 1.27)) hide)
-    )
-    (property "Part" "RC0402JR-070RL" (at 247.65 138.43 90)
-      (effects (font (size 1.27 1.27)) hide)
-    )
-    (property "JLCPCB Part#" "" (at 247.65 138.43 0)
-      (effects (font (size 1.27 1.27)) hide)
-    )
-    (property "LCSC Part #" "C17168" (at 247.65 138.43 0)
-      (effects (font (size 1.27 1.27)) hide)
-    )
-    (pin "1")
-    (pin "2")
-    (instances
-      (project "BLE_REMOTE"
-        (path "/3c7105d6-b2e1-4841-966d-0562ae88783f/df7514b4-387c-47b1-a1bd-e93660408c5b"
-          (reference "R25") (unit 1)
-        )
-        (path "/3c7105d6-b2e1-4841-966d-0562ae88783f/df7514b4-387c-47b1-a1bd-e93660408c5b/a095a39f-6b3f-4eb2-81ef-a7fa39c10239"
-          (reference "R23") (unit 1)
-        )
-        (path "/3c7105d6-b2e1-4841-966d-0562ae88783f/df7514b4-387c-47b1-a1bd-e93660408c5b/a0a15605-c20d-4158-a513-aa16071bb857"
-          (reference "R27") (unit 1)
-        )
-        (path "/3c7105d6-b2e1-4841-966d-0562ae88783f"
-          (reference "R31") (unit 1)
-        )
-      )
-      (project "Battery"
-        (path "/671d4de1-777a-48e9-9f3d-613423e17047"
-          (reference "R1") (unit 1)
-        )
-      )
-      (project "BLEC_power"
-        (path "/a7925ddf-5c61-458f-8a66-a1453f1c9b4d"
-          (reference "R25") (unit 1)
         )
       )
@@
         )
       )
-    )
-  )
-  (symbol (lib_id "Device:R") (at 223.52 139.7 0) (unit 1)
-    (in_bom yes) (on_board yes) (dnp no)
-    (property "Reference" "R25" (at 220.98 139.7 90)
-      (effects (font (size 1.27 1.27)))
-    )
-    (property "Value" "0R" (at 223.52 139.7 90)
-      (effects (font (size 1.27 1.27)))
-    )
-    (property "Footprint" "Resistor_SMD:R_0402_1005Metric_Pad0.72x0.64mm_HandSolder" (at 221.742 139.7 90)
-      (effects (font (size 1.27 1.27)) hide)
-    )
-    (property "Datasheet" "https://www.digikey.ca/en/products/detail/yageo/RC0402FR-07100KL/726526" (at 223.52 139.7 0)
-      (effects (font (size 1.27 1.27)) hide)
-    )
-    (property "Part" "RC0402JR-070RL" (at 223.52 139.7 90)
-      (effects (font (size 1.27 1.27)) hide)
-    )
-    (property "JLCPCB Part#" "" (at 223.52 139.7 0)
-      (effects (font (size 1.27 1.27)) hide)
-    )
-    (property "LCSC Part #" "C17168" (at 223.52 139.7 0)
-      (effects (font (size 1.27 1.27)) hide)
-    )
-    (pin "1")
-    (pin "2")
-    (instances
-      (project "BLE_REMOTE"
-        (path "/3c7105d6-b2e1-4841-966d-0562ae88783f/df7514b4-387c-47b1-a1bd-e93660408c5b"
-          (reference "R25") (unit 1)
-        )
-        (path "/3c7105d6-b2e1-4841-966d-0562ae88783f/df7514b4-387c-47b1-a1bd-e93660408c5b/a095a39f-6b3f-4eb2-81ef-a7fa39c10239"
-          (reference "R23") (unit 1)
-        )
-        (path "/3c7105d6-b2e1-4841-966d-0562ae88783f/df7514b4-387c-47b1-a1bd-e93660408c5b/a0a15605-c20d-4158-a513-aa16071bb857"
-          (reference "R27") (unit 1)
-        )
-        (path "/3c7105d6-b2e1-4841-966d-0562ae88783f"
-          (reference "R30") (unit 1)
-        )
-      )
-      (project "Battery"
-        (path "/671d4de1-777a-48e9-9f3d-613423e17047"
-          (reference "R1") (unit 1)
-        )
-      )
-      (project "BLEC_power"
-        (path "/a7925ddf-5c61-458f-8a66-a1453f1c9b4d"
-          (reference "R25") (unit 1)
-        )
-      )
