File: _Electrical/BLE_REMOTE/USBC.kicad_sch (KiCad schematic)
At the start: 3 parts, among them J1 USBC

Commit message: asdasat
Parts:
- added R25: 0R, Resistor_SMD:R_0402_1005Metric_Pad0.72x0.64mm_HandSolder, symbol Device:R
- R8, R9: LCSC Part # (none) -> C25905
Connections:
- net GND: now also R25.2; no longer J1.S1 (SHIELD), J1.S2 (SHIELD__1), J1.S3 (SHIELD__2), J1.S4 (SHIELD__3)
- new net SHIELD: J1.S1 (SHIELD), J1.S2 (SHIELD__1), J1.S3 (SHIELD__2), J1.S4 (SHIELD__3), R25.1
Other:
- moved on the sheet: R8, R9

Commit message: ordered from JLCPCB
Parts:
- removed R25: 0R, Resistor_SMD:R_0402_1005Metric_Pad0.72x0.64mm_HandSolder, symbol Device:R
Connections:
- net SHIELD is gone; now on net GND: J1.S1 (SHIELD), J1.S2 (SHIELD__1), J1.S3 (SHIELD__2), J1.S4 (SHIELD__3)
Changed lines of the file:
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@@
     (stroke (width 0) (type default))
   )
-  (wire (pts (xy 76.2 96.52) (xy 76.2 99.06))
+  (wire (pts (xy 76.2 96.52) (xy 76.2 110.49))
     (stroke (width 0) (type default))
   )
@@
     (stroke (width 0) (type default))
   )
-  (wire (pts (xy 76.2 106.68) (xy 76.2 110.49))
-    (stroke (width 0) (type default))
-  )
   (wire (pts (xy 88.9 66.04) (xy 88.9 68.58))
     (stroke (width 0) (type default))
@@
   (wire (pts (xy 85.09 91.44) (xy 85.09 93.98))
     (stroke (width 0) (type default))
-  )
-  (global_label "SHIELD" (shape input) (at 76.2 96.52 180) (fields_autoplaced)
-    (effects (font (size 1.27 1.27)) (justify right))
-    (property "Intersheetrefs" "${INTERSHEET_REFS}" (at 66.7023 96.52 0)
-      (effects (font (size 1.27 1.27)) (justify right) hide)
-    )
   )
   (netclass_flag "" (length 2.54) (shape round) (at 78.74 76.2 0) (fields_autoplaced)
@@
         )
       )
-    )
-  )
-  (symbol (lib_id "Device:R") (at 76.2 102.87 0) (unit 1)
-    (in_bom yes) (on_board yes) (dnp no)
-    (property "Reference" "R25" (at 73.66 102.87 90)
-      (effects (font (size 1.27 1.27)))
-    )
-    (property "Value" "0R" (at 76.2 102.87 90)
-      (effects (font (size 1.27 1.27)))
-    )
-    (property "Footprint" "Resistor_SMD:R_0402_1005Metric_Pad0.72x0.64mm_HandSolder" (at 74.422 102.87 90)
-      (effects (font (size 1.27 1.27)) hide)
-    )
-    (property "Datasheet" "https://www.digikey.ca/en/products/detail/yageo/RC0402FR-07100KL/726526" (at 76.2 102.87 0)
-      (effects (font (size 1.27 1.27)) hide)
-    )
-    (property "Part" "RC0402JR-070RL" (at 76.2 102.87 90)
-      (effects (font (size 1.27 1.27)) hide)
-    )
-    (property "JLCPCB Part#" "" (at 76.2 102.87 0)
-      (effects (font (size 1.27 1.27)) hide)
-    )
-    (property "LCSC Part #" "C17168" (at 76.2 102.87 0)
-      (effects (font (size 1.27 1.27)) hide)
-    )
-    (pin "1")
-    (pin "2")
-    (instances
-      (project "BLE_REMOTE"
-        (path "/3c7105d6-b2e1-4841-966d-0562ae88783f/df7514b4-387c-47b1-a1bd-e93660408c5b"
-          (reference "R25") (unit 1)
-        )
-        (path "/3c7105d6-b2e1-4841-966d-0562ae88783f/df7514b4-387c-47b1-a1bd-e93660408c5b/a095a39f-6b3f-4eb2-81ef-a7fa39c10239"
-          (reference "R23") (unit 1)
-        )
-        (path "/3c7105d6-b2e1-4841-966d-0562ae88783f/df7514b4-387c-47b1-a1bd-e93660408c5b/a0a15605-c20d-4158-a513-aa16071bb857"
-          (reference "R27") (unit 1)
-        )
-      )
-      (project "Battery"
-        (path "/671d4de1-777a-48e9-9f3d-613423e17047"
-          (reference "R1") (unit 1)
-        )
-      )
-      (project "BLEC_power"
-        (path "/a7925ddf-5c61-458f-8a66-a1453f1c9b4d"
-          (reference "R25") (unit 1)
-        )
-      )
